File: hw/arf154.sch (KiCad schematic (older format))
At the start: 0 parts

Commit message: USB connections made, need to add protection in VBUS power flag connection to avoid problems when not powered from USB
Parts:
- added R? (x2): 100K, 0603, symbol R_Small
Connections:
- net labels added: D+, D-, GND, VBUS, VBUS_DETECT, VCC
- wire segments 0 -> 13
Other:
- note added: "Main power circuit\n"
- note added: "Need to add protection"
- note added: "USB protection and connector\n"
Changed lines of the file:
@@
 $EndDescr
 $Sheet
-S 1000 2900 1350 2100
+S 800  3000 1250 4450
 U 55709F36
 F0 "MainProcessor" 60
 F1 "plugmodules/processing/atsamr21q1x.sch" 60
+F2 "PA0" I R 2050 3100 60
+F3 "PA1" I R 2050 3200 60
+F4 "PA2" I R 2050 3300 60
+F5 "PA3" I R 2050 3400 60
+F6 "PA4" I R 2050 3500 60
+F7 "PA5" I R 2050 3600 60
+F8 "PA6" I R 2050 3700 60
+F9 "PA7" I R 2050 3800 60
+F10 "PA8" I R 2050 3900 60
+F11 "PA9" I R 2050 4000 60
+F12 "PA12" I R 2050 4100 60
+F13 "PA13" I R 2050 4200 60
+F14 "PA14" I R 2050 4300 60
+F15 "PA15" I R 2050 4400 60
+F16 "PA16" I R 2050 4600 60
+F17 "PA17" I R 2050 4800 60
+F18 "PA18" I R 2050 4950 60
+F19 "PA19" I R 2050 5100 60
+F20 "PA22" I R 2050 5300 60
+F21 "PA23" I R 2050 5450 60
+F22 "PA24" I R 2050 5600 60
+F23 "PA25" I R 2050 5700 60
+F24 "PA27" I R 2050 5900 60
+F25 "PA28" I R 2050 6000 60
 $EndSheet
 $Sheet
-S 1050 800  1100 1050
+S 800  900  1100 1050
 U 55722354
 F0 "MainPower" 60
@@
 $EndSheet
 $Sheet
-S 4750 850  1050 1100
+S 6900 1050 900  750
 U 557215E4
 F0 "Sheet557215E3" 60
 F1 "plugmodules/comm/usb.sch" 60
+F2 "D+" I L 6900 1450 60
+F3 "D-" I L 6900 1550 60
+F4 "VBUS" I L 6900 1300 60
 $EndSheet
+Text Notes 850  2250 0    60   ~ 0
+Main power circuit\n
+Text Notes 6900 2000 0    60   ~ 0
+USB protection and connector\n
+Text Label 2200 5600 0    60   ~ 0
+D+
+Wire Wire Line
+	2200 5600 2050 5600
+Text Label 2200 5700 0    60   ~ 0
+D-
+Wire Wire Line
+	2050 5700 2200 5700
+Text Label 6750 1450 2    60   ~ 0
+D+
+Text Label 6750 1550 2    60   ~ 0
+D-
+Wire Wire Line
+	6750 1550 6900 1550
+Wire Wire Line
+	6750 1450 6900 1450
+$Comp
+L R_Small R?
+U 1 1 557DBA1C
+P 6200 1200
+F 0 "R?" H 6230 1220 50  0000 L CNN
+F 1 "100K" H 6230 1160 50  0000 L CNN
+F 2 "0603" H 6200 1200 60  0001 C CNN
+F 3 "" H 6200 1200 60  0000 C CNN
+	1    6200 1200
+	1    0    0    -1
+$EndComp
+$Comp
+L R_Small R?
+U 1 1 557DC4F8
+P 6200 1500
+F 0 "R?" H 6230 1520 50  0000 L CNN
+F 1 "100K" H 6230 1460 50  0000 L CNN
+F 2 "0603" H 6200 1500 60  0001 C CNN
+F 3 "" H 6200 1500 60  0000 C CNN
+	1    6200 1500
+	1    0    0    -1
+$EndComp
+Wire Wire Line
+	6200 1300 6200 1400
+$Comp
+L GND #PWR?
+U 1 1 557DC734
+P 6200 1700
+F 0 "#PWR?" H 6200 1450 50  0001 C CNN
+F 1 "GND" H 6200 1550 50  0000 C CNN
+F 2 "" H 6200 1700 60  0000 C CNN
+F 3 "" H 6200 1700 60  0000 C CNN
+	1    6200 1700
+	1    0    0    -1
+$EndComp
+Wire Wire Line
+	6200 1600 6200 1700
+Text Label 5950 1350 2    60   ~ 0
+VBUS_DETECT
+Text Label 6700 1300 2    60   ~ 0
+VBUS
+Wire Wire Line
+	6700 1300 6900 1300
+Text Label 6200 1000 2    60   ~ 0
+VBUS
+Wire Wire Line
+	6200 1000 6200 1100
+Wire Wire Line
+	5950 1350 6200 1350
+Connection ~ 6200 1350
+Text Label 2250 5450 0    60   ~ 0
+VBUS_DETECT
+Wire Wire Line
+	2050 5450 2250 5450
+Text Label 2650 950  2    60   ~ 0
+VBUS
+$Comp
+L VCC #PWR?
+U 1 1 557DE4B6
+P 3050 1000
+F 0 "#PWR?" H 3050 850 50  0001 C CNN
+F 1 "VCC" H 3050 1150 50  0000 C CNN
+F 2 "" H 3050 1000 60  0000 C CNN
+F 3 "" H 3050 1000 60  0000 C CNN
+	1    3050 1000
+	1    0    0    -1
+$EndComp
+Wire Wire Line
+	2650 950  2650 1100
+Wire Wire Line
+	2650 1100 3050 1100
+Wire Wire Line
+	3050 1100 3050 1000
+Text Notes 2400 1250 0    60   ~ 0
+Need to add protection
 $EndSCHEMATC

Commit message: First schematics done. Need to finish connections and add power separation of VBUS-VCC
Parts:
- added P? (x2): CONN_01X15, symbol CONN_01X15
Changed lines of the file:
@@
 Text Notes 2400 1250 0    60   ~ 0
 Need to add protection
+$Comp
+L CONN_01X15 P?
+U 1 1 557FE7ED
+P 8500 4200
+F 0 "P?" H 8500 5000 50  0000 C CNN
+F 1 "CONN_01X15" V 8600 4200 50  0000 C CNN
+F 2 "" H 8500 4200 60  0000 C CNN
+F 3 "" H 8500 4200 60  0000 C CNN
+	1    8500 4200
+	-1   0    0    -1
+$EndComp
+$Comp
+L CONN_01X15 P?
+U 1 1 557FE89D
+P 7150 4150
+F 0 "P?" H 7150 4950 50  0000 C CNN
+F 1 "CONN_01X15" V 7250 4150 50  0000 C CNN
+F 2 "" H 7150 4150 60  0000 C CNN
+F 3 "" H 7150 4150 60  0000 C CNN
+	1    7150 4150
+	1    0    0    -1
+$EndComp
 $EndSCHEMATC

Commit message: README update, Schematics almost done(need to finish power section)
Parts:
- P1, P2: renamed from P?; footprint (none) -> Pin_Headers:Pin_Header_Straight_1x15
- R1, R2: renamed from R?; footprint 0603 -> Resistors_SMD:R_0603_HandSoldering
Changed lines of the file:
@@
 $EndSheet
 $Sheet
-S 6900 1050 900  750
+S 5100 750  900  750
 U 557215E4
 F0 "Sheet557215E3" 60
 F1 "plugmodules/comm/usb.sch" 60
-F2 "D+" I L 6900 1450 60
-F3 "D-" I L 6900 1550 60
-F4 "VBUS" I L 6900 1300 60
+F2 "D+" I L 5100 1150 60
+F3 "D-" I L 5100 1250 60
+F4 "VBUS" I L 5100 1000 60
 $EndSheet
 Text Notes 850  2250 0    60   ~ 0
 Main power circuit\n
-Text Notes 6900 2000 0    60   ~ 0
+Text Notes 5100 1700 0    60   ~ 0
 USB protection and connector\n
 Text Label 2200 5600 0    60   ~ 0
@@
 Wire Wire Line
 	2050 5700 2200 5700
-Text Label 6750 1450 2    60   ~ 0
+Text Label 4950 1150 2    60   ~ 0
 D+
-Text Label 6750 1550 2    60   ~ 0
+Text Label 4950 1250 2    60   ~ 0
 D-
 Wire Wire Line
-	6750 1550 6900 1550
+	4950 1250 5100 1250
 Wire Wire Line
-	6750 1450 6900 1450
+	4950 1150 5100 1150
 $Comp
-L R_Small R?
+L R_Small R1
 U 1 1 557DBA1C
-P 6200 1200
-F 0 "R?" H 6230 1220 50  0000 L CNN
-F 1 "100K" H 6230 1160 50  0000 L CNN
-F 2 "0603" H 6200 1200 60  0001 C CNN
-F 3 "" H 6200 1200 60  0000 C CNN
-	1    6200 1200
+P 4400 900
+F 0 "R1" H 4430 920 50  0000 L CNN
+F 1 "100K" H 4430 860 50  0000 L CNN
+F 2 "Resistors_SMD:R_0603_HandSoldering" H 4400 900 60  0001 C CNN
+F 3 "" H 4400 900 60  0000 C CNN
+	1    4400 900
 	1    0    0    -1
 $EndComp
 $Comp
-L R_Small R?
+L R_Small R2
 U 1 1 557DC4F8
-P 6200 1500
-F 0 "R?" H 6230 1520 50  0000 L CNN
-F 1 "100K" H 6230 1460 50  0000 L CNN
-F 2 "0603" H 6200 1500 60  0001 C CNN
-F 3 "" H 6200 1500 60  0000 C CNN
-	1    6200 1500
+P 4400 1200
+F 0 "R2" H 4430 1220 50  0000 L CNN
+F 1 "100K" H 4430 1160 50  0000 L CNN
+F 2 "Resistors_SMD:R_0603_HandSoldering" H 4400 1200 60  0001 C CNN
+F 3 "" H 4400 1200 60  0000 C CNN
+	1    4400 1200
 	1    0    0    -1
 $EndComp
 Wire Wire Line
-	6200 1300 6200 1400
+	4400 1000 4400 1100
 $Comp
-L GND #PWR?
+L GND #PWR01
 U 1 1 557DC734
-P 6200 1700
-F 0 "#PWR?" H 6200 1450 50  0001 C CNN
-F 1 "GND" H 6200 1550 50  0000 C CNN
-F 2 "" H 6200 1700 60  0000 C CNN
-F 3 "" H 6200 1700 60  0000 C CNN
-	1    6200 1700
+P 4400 1400
+F 0 "#PWR01" H 4400 1150 50  0001 C CNN
+F 1 "GND" H 4400 1250 50  0000 C CNN
+F 2 "" H 4400 1400 60  0000 C CNN
+F 3 "" H 4400 1400 60  0000 C CNN
+	1    4400 1400
 	1    0    0    -1
 $EndComp
 Wire Wire Line
-	6200 1600 6200 1700
-Text Label 5950 1350 2    60   ~ 0
+	4400 1300 4400 1400
+Text Label 4150 1050 2    60   ~ 0
 VBUS_DETECT
-Text Label 6700 1300 2    60   ~ 0
+Text Label 4900 1000 2    60   ~ 0
 VBUS
 Wire Wire Line
-	6700 1300 6900 1300
-Text Label 6200 1000 2    60   ~ 0
+	4900 1000 5100 1000
+Text Label 4400 700  2    60   ~ 0
 VBUS
 Wire Wire Line
-	6200 1000 6200 1100
+	4400 700  4400 800
 Wire Wire Line
-	5950 1350 6200 1350
-Connection ~ 6200 1350
+	4150 1050 4400 1050
+Connection ~ 4400 1050
 Text Label 2250 5450 0    60   ~ 0
 VBUS_DETECT
@@
 VBUS
 $Comp
-L VCC #PWR?
+L VCC #PWR02
 U 1 1 557DE4B6
 P 3050 1000
-F 0 "#PWR?" H 3050 850 50  0001 C CNN
+F 0 "#PWR02" H 3050 850 50  0001 C CNN
 F 1 "VCC" H 3050 1150 50  0000 C CNN
 F 2 "" H 3050 1000 60  0000 C CNN
@@
 Need to add protection
 $Comp
-L CONN_01X15 P?
+L CONN_01X15 P2
 U 1 1 557FE7ED
-P 8500 4200
-F 0 "P?" H 8500 5000 50  0000 C CNN
-F 1 "CONN_01X15" V 8600 4200 50  0000 C CNN
-F 2 "" H 8500 4200 60  0000 C CNN
-F 3 "" H 8500 4200 60  0000 C CNN
-	1    8500 4200
+P 5700 4050
+F 0 "P2" H 5700 4850 50  0000 C CNN
+F 1 "CONN_01X15" V 5800 4050 50  0000 C CNN
+F 2 "Pin_Headers:Pin_Header_Straight_1x15" H 5700 4050 60  0001 C CNN
+F 3 "" H 5700 4050 60  0000 C CNN
+	1    5700 4050
 	-1   0    0    -1
 $EndComp
 $Comp
-L CONN_01X15 P?
+L CONN_01X15 P1
 U 1 1 557FE89D
-P 7150 4150
-F 0 "P?" H 7150 4950 50  0000 C CNN
-F 1 "CONN_01X15" V 7250 4150 50  0000 C CNN
-F 2 "" H 7150 4150 60  0000 C CNN
-F 3 "" H 7150 4150 60  0000 C CNN
-	1    7150 4150
+P 4350 4000
+F 0 "P1" H 4350 4800 50  0000 C CNN
+F 1 "CONN_01X15" V 4450 4000 50  0000 C CNN
+F 2 "Pin_Headers:Pin_Header_Straight_1x15" H 4350 4000 60  0001 C CNN
+F 3 "" H 4350 4000 60  0000 C CNN
+	1    4350 4000
 	1    0    0    -1
 $EndComp

Commit message: Started layout, minor gitignore modification
Parts:
- P1: value CONN_01X15 -> Cn1
- P2: value CONN_01X15 -> Cn2
Connections:
- net labels added: 5V, A0, A1, A2, A3, A4, A5, A6, A7, D10, D11, D12, D13, D2, D3, D4, D5, D6, D7, D8, D9, D_N, D_P, REF, RST, RX0, TX1, VDD, VIN
- net labels removed: D+, D-
- wire segments 13 -> 43
Changed lines of the file:
@@
 F24 "PA27" I R 2050 5900 60
 F25 "PA28" I R 2050 6000 60
+F26 "RST" I R 2050 6400 60
 $EndSheet
 $Sheet
@@
 USB protection and connector\n
 Text Label 2200 5600 0    60   ~ 0
-D+
+D_P
 Wire Wire Line
 	2200 5600 2050 5600
 Text Label 2200 5700 0    60   ~ 0
-D-
+D_N
 Wire Wire Line
 	2050 5700 2200 5700
 Text Label 4950 1150 2    60   ~ 0
-D+
+D_P
 Text Label 4950 1250 2    60   ~ 0
-D-
+D_N
 Wire Wire Line
 	4950 1250 5100 1250
@@
 L CONN_01X15 P2
 U 1 1 557FE7ED
-P 5700 4050
-F 0 "P2" H 5700 4850 50  0000 C CNN
-F 1 "CONN_01X15" V 5800 4050 50  0000 C CNN
-F 2 "Pin_Headers:Pin_Header_Straight_1x15" H 5700 4050 60  0001 C CNN
-F 3 "" H 5700 4050 60  0000 C CNN
-	1    5700 4050
+P 5150 4000
+F 0 "P2" H 5150 4800 50  0000 C CNN
+F 1 "Cn2" V 5250 4000 50  0000 C CNN
+F 2 "Pin_Headers:Pin_Header_Straight_1x15" H 5150 4000 60  0001 C CNN
+F 3 "" H 5150 4000 60  0000 C CNN
+	1    5150 4000
 	-1   0    0    -1
 $EndComp
@@
 P 4350 4000
 F 0 "P1" H 4350 4800 50  0000 C CNN
-F 1 "CONN_01X15" V 4450 4000 50  0000 C CNN
+F 1 "Cn1" V 4450 4000 50  0000 C CNN
 F 2 "Pin_Headers:Pin_Header_Straight_1x15" H 4350 4000 60  0001 C CNN
 F 3 "" H 4350 4000 60  0000 C CNN
@@
 	1    0    0    -1
 $EndComp
+Text Label 2300 6400 0    60   ~ 0
+RST
+Wire Wire Line
+	2050 6400 2300 6400
+Text Label 4000 3500 2    60   ~ 0
+RST
+$Comp
+L GND #PWR03
+U 1 1 5582A053
+P 3900 3600
+F 0 "#PWR03" H 3900 3350 50  0001 C CNN
+F 1 "GND" H 3900 3450 50  0000 C CNN
+F 2 "" H 3900 3600 60  0000 C CNN
+F 3 "" H 3900 3600 60  0000 C CNN
+	1    3900 3600
+	0    1    1    0
+$EndComp
+$Comp
+L GND #PWR04
+U 1 1 5582A221
+P 5600 3400
+F 0 "#PWR04" H 5600 3150 50  0001 C CNN
+F 1 "GND" H 5600 3250 50  0000 C CNN
+F 2 "" H 5600 3400 60  0000 C CNN
+F 3 "" H 5600 3400 60  0000 C CNN
+	1    5600 3400
+	0    -1   -1   0
+$EndComp
+Wire Wire Line
+	5350 3400 5600 3400
+Wire Wire Line
+	4000 3500 4150 3500
+Wire Wire Line
+	3900 3600 4150 3600
+Text Label 5450 3300 0    60   ~ 0
+VIN
+Wire Wire Line
+	5350 3300 5450 3300
+Text Label 4000 3300 2    60   ~ 0
+TX1
+Text Label 4000 3400 2    60   ~ 0
+RX0
+Text Label 4000 3700 2    60   ~ 0
+D2
+Text Label 4000 3800 2    60   ~ 0
+D3
+Text Label 4000 3900 2    60   ~ 0
+D4
+Text Label 4000 4000 2    60   ~ 0
+D5
+Text Label 4000 4100 2    60   ~ 0
+D6
+Wire Wire Line
+	4000 3300 4150 3300
+Wire Wire Line
+	4000 3400 4150 3400
+Wire Wire Line
+	4000 3700 4150 3700
+Wire Wire Line
+	4000 3800 4150 3800
+Wire Wire Line
+	4000 3900 4150 3900
+Wire Wire Line
+	4000 4000 4150 4000
+Wire Wire Line
+	4000 4100 4150 4100
+Text Label 4000 4200 2    60   ~ 0
+D7
+Text Label 4000 4300 2    60   ~ 0
+D8
+Text Label 4000 4400 2    60   ~ 0
+D9
+Text Label 4000 4500 2    60   ~ 0
+D10
+Text Label 4000 4600 2    60   ~ 0
+D11
+Text Label 4000 4700 2    60   ~ 0
+D12
+Wire Wire Line
+	4000 4700 4150 4700
+Wire Wire Line
+	4000 4600 4150 4600
+Wire Wire Line
+	4000 4500 4150 4500
+Wire Wire Line
+	4150 4400 4000 4400
+Wire Wire Line
+	4000 4300 4150 4300
+Wire Wire Line
+	4150 4200 4000 4200
+Text Label 5450 4700 0    60   ~ 0
+D13
+Wire Wire Line
+	5450 4700 5350 4700
+Text Label 5450 4500 0    60   ~ 0
+REF
+Text Label 5450 4400 0    60   ~ 0
+A0
+Text Label 5450 4300 0    60   ~ 0
+A1
+Text Label 5450 4200 0    60   ~ 0
+A2
+Text Label 5450 4100 0    60   ~ 0
+A3
+Text Label 5450 4000 0    60   ~ 0
+A4
+Text Label 5450 3900 0    60   ~ 0
+A5
+Text Label 5450 3800 0    60   ~ 0
+A6
+Text Label 5450 3700 0    60   ~ 0
+A7
+Text Label 5450 3600 0    60   ~ 0
+5V
+Text Label 5450 3500 0    60   ~ 0
+RST
+Wire Wire Line
+	5350 3500 5450 3500
+Wire Wire Line
+	5450 3600 5350 3600
+Wire Wire Line
+	5350 3700 5450 3700
+Wire Wire Line
+	5450 3800 5350 3800
+Wire Wire Line
+	5350 3900 5450 3900
+Wire Wire Line
+	5350 4000 5450 4000
+Wire Wire Line
+	5350 4100 5450 4100
+Wire Wire Line
+	5350 4200 5450 4200
+Wire Wire Line
+	5350 4400 5450 4400
+Wire Wire Line
+	5350 4500 5450 4500
+$Comp
+L VDD #PWR05
+U 1 1 5583100F
+P 5600 4600
+F 0 "#PWR05" H 5600 4450 50  0001 C CNN
+F 1 "VDD" H 5600 4750 50  0000 C CNN
+F 2 "" H 5600 4600 60  0000 C CNN
+F 3 "" H 5600 4600 60  0000 C CNN
+	1    5600 4600
+	0    1    1    0
+$EndComp
+Wire Wire Line
+	5350 4600 5600 4600
 $EndSCHEMATC

Commit message: Schematics change for a smaller regulator, added a new sch module, layout update
Changed lines of the file:
@@
 EESchema Schematic File Version 2
+LIBS:arf154-rescue
 LIBS:power
 LIBS:device
@@
 U 55722354
 F0 "MainPower" 60
-F1 "plugmodules/power/linear3v3.sch" 60
+F1 "plugmodules/power/linear3v3small.sch" 60
 $EndSheet
 $Sheet

Commit message: Layout update, footprint changed to 0402, atsam component fix
Parts:
- R1, R2: footprint Resistors_SMD:R_0603_HandSoldering -> Resistors_SMD:R_0402
Connections:
- wire segments 43 -> 52
Changed lines of the file:
@@
 $EndDescr
-$Sheet
-S 800  3000 1250 4450
-U 55709F36
-F0 "MainProcessor" 60
-F1 "plugmodules/processing/atsamr21q1x.sch" 60
-F2 "PA0" I R 2050 3100 60
-F3 "PA1" I R 2050 3200 60
-F4 "PA2" I R 2050 3300 60
-F5 "PA3" I R 2050 3400 60
-F6 "PA4" I R 2050 3500 60
-F7 "PA5" I R 2050 3600 60
-F8 "PA6" I R 2050 3700 60
-F9 "PA7" I R 2050 3800 60
-F10 "PA8" I R 2050 3900 60
-F11 "PA9" I R 2050 4000 60
-F12 "PA12" I R 2050 4100 60
-F13 "PA13" I R 2050 4200 60
-F14 "PA14" I R 2050 4300 60
-F15 "PA15" I R 2050 4400 60
-F16 "PA16" I R 2050 4600 60
-F17 "PA17" I R 2050 4800 60
-F18 "PA18" I R 2050 4950 60
-F19 "PA19" I R 2050 5100 60
-F20 "PA22" I R 2050 5300 60
-F21 "PA23" I R 2050 5450 60
-F22 "PA24" I R 2050 5600 60
-F23 "PA25" I R 2050 5700 60
-F24 "PA27" I R 2050 5900 60
-F25 "PA28" I R 2050 6000 60
-F26 "RST" I R 2050 6400 60
-$EndSheet
 $Sheet
 S 800  900  1100 1050
@@
 F 0 "R1" H 4430 920 50  0000 L CNN
 F 1 "100K" H 4430 860 50  0000 L CNN
-F 2 "Resistors_SMD:R_0603_HandSoldering" H 4400 900 60  0001 C CNN
+F 2 "Resistors_SMD:R_0402" H 4400 900 60  0001 C CNN
 F 3 "" H 4400 900 60  0000 C CNN
 	1    4400 900
@@
 F 0 "R2" H 4430 1220 50  0000 L CNN
 F 1 "100K" H 4430 1160 50  0000 L CNN
-F 2 "Resistors_SMD:R_0603_HandSoldering" H 4400 1200 60  0001 C CNN
+F 2 "Resistors_SMD:R_0402" H 4400 1200 60  0001 C CNN
 F 3 "" H 4400 1200 60  0000 C CNN
 	1    4400 1200
@@
 Wire Wire Line
 	5350 4600 5600 4600
+Wire Wire Line
+	5350 4300 5450 4300
+Text Label 2150 4050 0    60   ~ 0
+A0
+Text Label 2150 3950 0    60   ~ 0
+A1
+Text Label 2150 3850 0    60   ~ 0
+A2
+Text Label 2150 3750 0    60   ~ 0
+A3
+Text Label 2150 3350 0    60   ~ 0
+A4
+Text Label 2150 3450 0    60   ~ 0
+A5
+Text Label 2150 3550 0    60   ~ 0
+A6
+Text Label 2150 3650 0    60   ~ 0
+A7
+$Sheet
+S 800  3000 1250 4450
+U 55709F36
+F0 "MainProcessor" 60
+F1 "plugmodules/processing/atsamr21q1x.sch" 60
+F2 "PA0" I R 2050 3100 60
+F3 "PA1" I R 2050 3200 60
+F4 "PA4" I R 2050 3350 60
+F5 "PA5" I R 2050 3450 60
+F6 "PA6" I R 2050 3550 60
+F7 "PA7" I R 2050 3650 60
+F8 "PA8" I R 2050 3750 60
+F9 "PA9" I R 2050 3850 60
+F10 "PA12" I R 2050 4500 60
+F11 "PA13" I R 2050 4200 60
+F12 "PA14" I R 2050 4300 60
+F13 "PA15" I R 2050 4400 60
+F14 "PA16" I R 2050 4600 60
+F15 "PA17" I R 2050 4800 60
+F16 "PA18" I R 2050 4950 60
+F17 "PA19" I R 2050 5100 60
+F18 "PA22" I R 2050 5300 60
+F19 "PA23" I R 2050 5450 60
+F20 "PA24" I R 2050 5600 60
+F21 "PA25" I R 2050 5700 60
+F22 "PA27" I R 2050 5900 60
+F23 "PA28" I R 2050 6000 60
+F24 "RST" I R 2050 6400 60
+F25 "PB2" I R 2050 3950 60
+F26 "PB3" I R 2050 4050 60
+$EndSheet
+Wire Wire Line
+	2050 3350 2150 3350
+Wire Wire Line
+	2150 3450 2050 3450
+Wire Wire Line
+	2050 3550 2150 3550
+Wire Wire Line
+	2150 3650 2050 3650
+Wire Wire Line
+	2050 3750 2150 3750
+Wire Wire Line
+	2150 3850 2050 3850
+Wire Wire Line
+	2050 3950 2150 3950
+Wire Wire Line
+	2150 4050 2050 4050
 $EndSCHEMATC

Commit message: Layout for the analog pads and DRC fix on the USB signals
Changed lines of the file:
@@
 Wire Wire Line
 	5350 4300 5450 4300
+Text Label 2150 3950 0    60   ~ 0
+A0
 Text Label 2150 4050 0    60   ~ 0
-A0
-Text Label 2150 3950 0    60   ~ 0
 A1
+Text Label 2150 3350 0    60   ~ 0
+A2
+Text Label 2150 3450 0    60   ~ 0
+A3
+Text Label 2150 3550 0    60   ~ 0
+A4
+Text Label 2150 3650 0    60   ~ 0
+A5
+Text Label 2150 3750 0    60   ~ 0
+A6
 Text Label 2150 3850 0    60   ~ 0
-A2
-Text Label 2150 3750 0    60   ~ 0
-A3
-Text Label 2150 3350 0    60   ~ 0
-A4
-Text Label 2150 3450 0    60   ~ 0
-A5
-Text Label 2150 3550 0    60   ~ 0
-A6
-Text Label 2150 3650 0    60   ~ 0
 A7
 $Sheet
