File: hw/arf154.sch (KiCad schematic (older format))
At the start: 4 parts, among them P1 Cn1, P2 Cn2

Commit message: Layout modifications
Parts:
- added D2, D3: D_Small, symbol D_Small
Connections:
- wire segments 52 -> 57
Other:
- note removed: "Need to add protection"
Changed lines of the file:
@@
 	2650 950  2650 1100
 Wire Wire Line
-	2650 1100 3050 1100
-Wire Wire Line
 	3050 1100 3050 1000
-Text Notes 2400 1250 0    60   ~ 0
-Need to add protection
 $Comp
 L CONN_01X15 P2
@@
 Wire Wire Line
 	2150 4050 2050 4050
+$Comp
+L D_Small D2
+U 1 1 559A6648
+P 2850 1100
+F 0 "D2" H 2800 1180 50  0000 L CNN
+F 1 "D_Small" H 2700 1020 50  0000 L CNN
+F 2 "" V 2850 1100 60  0001 C CNN
+F 3 "" V 2850 1100 60  0000 C CNN
+	1    2850 1100
+	-1   0    0    1
+$EndComp
+Wire Wire Line
+	2650 1100 2750 1100
+Wire Wire Line
+	2950 1100 3050 1100
+$Comp
+L VCC #PWR06
+U 1 1 559A7350
+P 3050 1400
+F 0 "#PWR06" H 3050 1250 50  0001 C CNN
+F 1 "VCC" H 3050 1550 50  0000 C CNN
+F 2 "" H 3050 1400 60  0000 C CNN
+F 3 "" H 3050 1400 60  0000 C CNN
+	1    3050 1400
+	1    0    0    -1
+$EndComp
+Wire Wire Line
+	3050 1500 3050 1400
+$Comp
+L D_Small D3
+U 1 1 559A7357
+P 2850 1500
+F 0 "D3" H 2800 1580 50  0000 L CNN
+F 1 "D_Small" H 2700 1420 50  0000 L CNN
+F 2 "" V 2850 1500 60  0001 C CNN
+F 3 "" V 2850 1500 60  0000 C CNN
+	1    2850 1500
+	-1   0    0    1
+$EndComp
+Wire Wire Line
+	2950 1500 3050 1500
+Text Label 2650 1300 2    60   ~ 0
+VIN
+Wire Wire Line
+	2650 1300 2650 1500
+Wire Wire Line
+	2650 1500 2750 1500
 $EndSCHEMATC
